Commit message: fix: add fixed base to prevent OP3 from falling

File: ros2_control/op3_with_control.urdf.xacro (robot description, xacro)
@@ -1,4 +1,10 @@
 <?xml version="1.0"?>
 <robot xmlns:xacro="http://ros.org/wiki/xacro" name="robotis_op3">
+  <link name="world"/>
+  <joint name="base_fixed" type="fixed">
+    <parent link="world"/>
+    <child link="base_link"/>
+    <origin xyz="0 0 0.35" rpy="0 0 0"/>
+  </joint>
   <xacro:arg name="controller_config_file" default="forward_command_config.yaml"/>
   <xacro:include filename="$(find op3_description)/urdf/robotis_op3.urdf.xacro"/>

Commit message: base fixed

File: ros2_control/op3_with_control.urdf.xacro (robot description, xacro)
@@ -2,5 +2,5 @@
 <robot xmlns:xacro="http://ros.org/wiki/xacro" name="robotis_op3">
   <link name="world"/>
-  <joint name="base_fixed" type="fixed">
+  <joint name="world_to_op3_base" type="fixed">
     <parent link="world"/>
     <child link="base_link"/>

Commit message: fix

File: ros2_control/op3_with_control.urdf.xacro (robot description, xacro)
@@ -4,5 +4,5 @@
   <joint name="world_to_op3_base" type="fixed">
     <parent link="world"/>
-    <child link="base_link"/>
+    <child link="base"/>
     <origin xyz="0 0 0.35" rpy="0 0 0"/>
   </joint>
