Commit message: Fix fwd axis, standing pose values, and spawn height
- retargeting: fix body frame fwd vector — was cross(right,up)=+z=BEHIND
  person, now cross(up,right)=-z=toward camera. Fixes all pitch directions.
- retargeting: update STANDING_DEFAULTS to official OP3 values (π/6,π/3,π/6)
- xacro: match initial_value to official OP3 standing pose (0.5236/1.0472)
- urdf.xacro + launch: lower spawn z from 0.35 → 0.31m (official pelvis height)

Co-Authored-By: Claude Sonnet 4.6 <noreply@anthropic.com>

File: ros2_control/op3_ros2_control.xacro (robot description, xacro)
@@ -58,30 +58,30 @@
       <joint name="l_hip_pitch">
         <command_interface name="position"/>
-        <state_interface name="position"><param name="initial_value">-0.57</param></state_interface>
+        <state_interface name="position"><param name="initial_value">-0.5236</param></state_interface>
         <state_interface name="velocity"><param name="initial_value">0.0</param></state_interface>
       </joint>
       <joint name="r_hip_pitch">
         <command_interface name="position"/>
-        <state_interface name="position"><param name="initial_value">0.57</param></state_interface>
+        <state_interface name="position"><param name="initial_value">0.5236</param></state_interface>
         <state_interface name="velocity"><param name="initial_value">0.0</param></state_interface>
       </joint>
       <joint name="l_knee">
         <command_interface name="position"/>
-        <state_interface name="position"><param name="initial_value">1.2</param></state_interface>
+        <state_interface name="position"><param name="initial_value">1.0472</param></state_interface>
         <state_interface name="velocity"><param name="initial_value">0.0</param></state_interface>
       </joint>
       <joint name="r_knee">
         <command_interface name="position"/>
-        <state_interface name="position"><param name="initial_value">1.2</param></state_interface>
+        <state_interface name="position"><param name="initial_value">1.0472</param></state_interface>
         <state_interface name="velocity"><param name="initial_value">0.0</param></state_interface>
       </joint>
       <joint name="l_ank_pitch">
         <command_interface name="position"/>
-        <state_interface name="position"><param name="initial_value">0.62</param></state_interface>
+        <state_interface name="position"><param name="initial_value">0.5236</param></state_interface>
         <state_interface name="velocity"><param name="initial_value">0.0</param></state_interface>
       </joint>
       <joint name="r_ank_pitch">
         <command_interface name="position"/>
-        <state_interface name="position"><param name="initial_value">-0.62</param></state_interface>
+        <state_interface name="position"><param name="initial_value">-0.5236</param></state_interface>
         <state_interface name="velocity"><param name="initial_value">0.0</param></state_interface>
       </joint>

File: ros2_control/op3_with_control.urdf.xacro (robot description, xacro)
@@ -5,5 +5,5 @@
     <parent link="world"/>
     <child link="base"/>
-    <origin xyz="0 0 0.35" rpy="0 0 0"/>
+    <origin xyz="0 0 0.31" rpy="0 0 0"/>
   </joint>
   <xacro:arg name="controller_config_file" default="forward_command_config.yaml"/>
